File: cga_pm_alice/cga_pm_alice.sch (KiCad schematic (older format))
At the start: 197 parts, among them J1 MX-LED, K1 MX-LED, M1 MX-LED, P1 MX-LED, Q1 MX-LED, SW1 reset_button, T1 MX-LED, U1 MX-LED, X1 MX-LED, Y1 MX-LED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

Commit message: Trying the ZigZag PM footprint
Parts:
- PM1: footprint Keebio-Parts:ArduinoProMicro -> Keebio-Parts:ArduinoProMicro-ZigZag
Changed lines of the file:
@@
 F 0 "PM1" H 9150 2537 60  0000 C CNN
 F 1 "ProMicro" H 9150 2431 60  0000 C CNN
-F 2 "Keebio-Parts:ArduinoProMicro" V 10200 -800 60  0001 C CNN
+F 2 "Keebio-Parts:ArduinoProMicro-ZigZag" V 10200 -800 60  0001 C CNN
 F 3 "" V 10200 -800 60  0001 C CNN
 	1    9150 1700
