File: cga_proto_boards/cga_proto_boards.sch (KiCad schematic (older format))
At the start: 14 parts, among them Q1 2N7002, T1 TRRS, U1 Elite-C

Commit message: Finalize v1 of the sideways cga proto board
Parts:
- removed H1: LEDsOut, Keebio-Parts:SinglePad, symbol keebio:Hole
- removed H2: RGB, Keebio-Parts:SinglePad, symbol keebio:Hole
- removed H3: GND, Keebio-Parts:SinglePad, symbol keebio:Hole
- removed H4: VCC, Keebio-Parts:SinglePad, symbol keebio:Hole
- added H1: LEDs, Keebio-Parts:SinglePad, symbol Mechanical:MountingHole_Pad
- added H2: GND, Keebio-Parts:SinglePad, symbol Mechanical:MountingHole_Pad
- added H3: VCC, Keebio-Parts:SinglePad, symbol Mechanical:MountingHole_Pad
- added J1, J2: 3_way_jumper, Keebio-Parts:3_way_solder_jumper, symbol keebio:3_way_jumper
- added Q2: 2N7002, Keebio-Parts:SOT-23_Handsoldering, symbol Transistor_FET:2N7002
- added RT1, RT2: 4.7k, Keebio-Parts:Resistor-2-sided, symbol Device:R_Small
- RQ1: footprint Keebio-Parts:Resistor-Hybrid-Back -> Keebio-Parts:Resistor-2-sided
- Reset1: footprint Keebio-Parts:SW_Tactile_SPST_Angled_MJTP1117 -> Keebio-Parts:SW_Two_sided
Connections:
- net SCL-SCK is gone; now on net SCL: O1.3 (SCK), O2.3 (SCK)
- net GND: now also H2.1, Q2.2 (S)
- net LEDs: now also Q2.1 (G)
- net LEDsOut: now also H1.1, Q2.3 (D)
- net SCL: now also J1.1 (Input1)
- net SDA: now also J2.1 (Input1)
- net TRRS1: now also J1.2 (Output), RT2.2; no longer Cs1.1 (P1), U1.1 (TX0/PD3)
- net TRRS2: now also J2.2 (Output), RT1.2; no longer Cs1.2 (P2), U1.2 (RX1/PD2)
- net VCC: now also H3.1, RT1.1, RT2.1
- new net RX: Cs1.2 (P2), J1.3 (Input2), U1.2 (RX1/PD2)
- new net TX: Cs1.1 (P1), J2.3 (Input2), U1.1 (TX0/PD3)
Other:
- moved on the sheet: RQ1
